Commit message: 部署成功

File: deploy_cpp/robot/mybot_v2_1/urdf/mybot_v2_1.urdf (robot description, URDF)
Before this commit: robot mybot_v2_1, 18 links, 17 joints
Links:
- link FL_calf: geometry collision box size=0.03 0.05 0.2; visual mesh filename=package://deploy_cpp/robot/mybot_v2_1/meshes/FL_calf.STL
- link FL_foot: geometry collision sphere radius=0.02; visual mesh filename=package://deploy_cpp/robot/mybot_v2_1/meshes/FL_foot.STL
- link FL_hip: geometry collision cylinder length=0.05 radius=0.05; visual mesh filename=package://deploy_cpp/robot/mybot_v2_1/meshes/FL_hip.STL
- link FL_thigh: geometry collision box size=0.04 0.04 0.2; visual mesh filename=package://deploy_cpp/robot/mybot_v2_1/meshes/FL_thigh.STL
- link FR_calf: geometry collision box size=0.03 0.05 0.2; visual mesh filename=package://deploy_cpp/robot/mybot_v2_1/meshes/FR_calf.STL
- link FR_foot: geometry collision sphere radius=0.02; visual mesh filename=package://deploy_cpp/robot/mybot_v2_1/meshes/FR_foot.STL
- link FR_hip: geometry collision cylinder length=0.05 radius=0.05; visual mesh filename=package://deploy_cpp/robot/mybot_v2_1/meshes/FR_hip.STL
- link FR_thigh: geometry collision box size=0.04 0.04 0.2; visual mesh filename=package://deploy_cpp/robot/mybot_v2_1/meshes/FR_thigh.STL
- link RL_calf: geometry collision box size=0.03 0.05 0.2; visual mesh filename=package://deploy_cpp/robot/mybot_v2_1/meshes/RL_calf.STL
- link RL_foot: geometry collision sphere radius=0.02; visual mesh filename=package://deploy_cpp/robot/mybot_v2_1/meshes/RL_foot.STL
- link RL_hip: geometry collision cylinder length=0.05 radius=0.05; visual mesh filename=package://deploy_cpp/robot/mybot_v2_1/meshes/RL_hip.STL
- link RL_thigh: geometry collision box size=0.04 0.04 0.2; visual mesh filename=package://deploy_cpp/robot/mybot_v2_1/meshes/RL_thigh.STL
- link RR_calf: geometry collision box size=0.03 0.05 0.2; visual mesh filename=package://deploy_cpp/robot/mybot_v2_1/meshes/RR_calf.STL
- link RR_foot: geometry collision sphere radius=0.02; visual mesh filename=package://deploy_cpp/robot/mybot_v2_1/meshes/RR_foot.STL
- link RR_hip: geometry collision cylinder length=0.05 radius=0.05; visual mesh filename=package://deploy_cpp/robot/mybot_v2_1/meshes/RR_hip.STL
- link RR_thigh: geometry collision box size=0.04 0.04 0.2; visual mesh filename=package://deploy_cpp/robot/mybot_v2_1/meshes/RR_thigh.STL
- link body: geometry collision box size=0.30 0.22 0.16; visual mesh filename=package://deploy_cpp/robot/mybot_v2_1/meshes/body.STL
