Commit message: 给urdf上额外加1kg载荷

File: resources/robots/mybot_v3/urdf/mybot_v3.urdf (robot description, URDF)
Before this commit: robot mybot_v3, 18 links, 17 joints
Links:
- added link payload_link, mass 1.0
Joints:
- added joint payload_joint: type fixed, parent body, child payload_link, origin xyz=0 0 0 rpy=0 0 0

Commit message: 更新RR_calf的质量和惯性参数

File: resources/robots/mybot_v3/urdf/mybot_v3.urdf (robot description, URDF)
Before this commit: robot mybot_v3, 19 links, 18 joints
Links:
- link RR_calf: mass 0.25719862 -> 0.23880158
