Commit message: Update mybot_v3 inertial properties

File: deploy_cpp/robot/mybot_v3/urdf/mybot_v3.urdf (robot description, URDF)
Before this commit: robot mybot_v3, 18 links, 17 joints
Links:
- link FR_calf: mass 0.23765586 -> 0.23708419
- link RR_calf: mass 0.25719862 -> 0.23880158
- link RR_thigh: mass 1.42118841 -> 1.45068546

File: resources/robots/mybot_v3/urdf/mybot_v3.urdf (robot description, URDF)
Before this commit: robot mybot_v3, 19 links, 18 joints
Links:
- link FR_calf: mass 0.23765586 -> 0.23708419
- link RR_thigh: mass 1.42118841 -> 1.45068546

File: resources/robots/mybot_v3_with_arm/urdf/mybot_v3_with_arm.urdf (robot description, URDF)
Before this commit: robot mybot_v3_with_arm, 19 links, 18 joints
Links:
- link FL_calf: mass 0.23708 -> 0.23708419
- link FL_hip: mass 0.88715 -> 0.88715151
- link FL_thigh: mass 1.4406 -> 1.44059854
- link FR_calf: mass 0.23708 -> 0.23708419
- link FR_hip: mass 0.88715 -> 0.88715151
- link FR_thigh: mass 1.4406 -> 1.44059854
- link RL_calf: mass 0.23708 -> 0.23880158
- link RL_hip: mass 0.88715 -> 0.88715151
- link RL_thigh: mass 1.4406 -> 1.45185979
- link RR_calf: mass 0.23708 -> 0.23880158
- link RR_hip: mass 0.88715 -> 0.88715151
- link RR_thigh: mass 1.4406 -> 1.45068546

Commit message: Update mybot_v3 inertial properties from revised data

File: deploy_cpp/robot/mybot_v3/urdf/mybot_v3.urdf (robot description, URDF)
Before this commit: robot mybot_v3, 18 links, 17 joints
Links:
- link FL_thigh: mass 1.44059854 -> 1.42386939
- link FR_thigh: mass 1.44059854 -> 1.42386939
- link RL_thigh: mass 1.45185979 -> 1.43392711
- link RR_calf: mass 0.23880158 -> 0.22489484
- link RR_thigh: mass 1.45068546 -> 1.40325573

File: resources/robots/mybot_v3/urdf/mybot_v3.urdf (robot description, URDF)
Before this commit: robot mybot_v3, 19 links, 18 joints
Links:
- link FL_thigh: mass 1.44059854 -> 1.42386939
- link FR_thigh: mass 1.44059854 -> 1.42386939
- link RL_thigh: mass 1.45185979 -> 1.43392711
- link RR_calf: mass 0.23880158 -> 0.22489484
- link RR_thigh: mass 1.45068546 -> 1.40325573

File: resources/robots/mybot_v3_with_arm/urdf/mybot_v3_with_arm.urdf (robot description, URDF)
Before this commit: robot mybot_v3_with_arm, 19 links, 18 joints
Links:
- link FL_thigh: mass 1.44059854 -> 1.42386939
- link FR_thigh: mass 1.44059854 -> 1.42386939
- link RL_thigh: mass 1.45185979 -> 1.43392711
- link RR_calf: mass 0.23880158 -> 0.22489484
- link RR_thigh: mass 1.45068546 -> 1.40325573
